File: KiCad/rp2040.kicad_sch (KiCad schematic)
At the start: 28 parts, among them U4 AP2112K-3.3, U5 GD25Q16xS, U6 RP2040, Y1 XYDBPCNANF-12MHZ

Commit message: update
Parts:
- U6: footprint beepberry:QFN-56-1EP_7x7mm_P0.4mm_EP5.6x5.6mm -> beepy:QFN-56-1EP_7x7mm_P0.4mm_EP5.6x5.6mm
